File: pcb-guide.kicad_sch (KiCad schematic)
At the start: 14 parts

Commit message: footprint
Parts:
- added D1, D2, D3, D4: D_Small, Diode_SMD:D_0805_2012Metric, symbol Device:D_Small
- added F1: 500mA, Fuse:Fuse_1206_3216Metric, symbol Device:Polyfuse
- added MX1, MX2, MX3, MX4: MX-NoLED, MX_Alps_Hybrid:MX-1U-NoLED, symbol MX_Alps_Hybrid:MX-NoLED
- added USB1: Molex-0548190589, random-keyboard-parts:Molex-0548190589, symbol random-keyboard-parts:Molex-0548190589
- C1, C2, C3, C4, C5, C6, C7: renamed from C?; footprint (none) -> Capacitor_SMD:C_0805_2012Metric
- R1, R2, R3, R4: renamed from R?; footprint (none) -> Resistor_SMD:R_0805_2012Metric
- SW1: renamed from SW?; footprint (none) -> random-keyboard-parts:SKQG-1155865
- Y1: renamed from Y?; footprint (none) -> Package_QFP:TQFP-44_10x10mm_P0.8mm
- gave numbers to parts that had none: 1
Connections:
- net +5V: now also F1.2
- net D+: now also USB1.3 (D+)
- net D-: now also USB1.4 (D-)
- net GND: now also USB1.1 (GND)
- net COL1: now reaches U1.28 (PB4)
- net COL1: now also MX2.1 (COL), MX4.1 (COL)
- net COL0: now reaches U1.29 (PB5)
- net COL0: now also MX1.1 (COL), MX3.1 (COL)
- net ROW1: now reaches U1.30 (PB6)
- net ROW1: now also D3.1 (K), D4.1 (K)
- new net: D3.2 (A), MX3.2 (ROW)
- new net: D1.2 (A), MX1.2 (ROW)
- new net: D4.2 (A), MX4.2 (ROW)
- new net: D2.2 (A), MX2.2 (ROW)
- new net ROW0: D1.1 (K), D2.1 (K)
- new net VCC: F1.1, USB1.5 (VBUS)

Commit message: save
Connections:
- net ROW0: now also U1.12 (PB7)
Changed lines of the file:
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@@
+    )
+  )
+  (global_label "ROW0" (shape input) (at 128.27 66.04 0) (fields_autoplaced)
+    (effects (font (size 1.27 1.27)) (justify left))
+    (property "Intersheet References" "${INTERSHEET_REFS}" (id 0) (at 135.9445 65.9606 0)
+      (effects (font (size 1.27 1.27)) (justify left) hide)
     )
   )
